Commit message: Implemented joystick control

File: description/main_core.xacro (robot description, xacro)
@@ -44,4 +44,6 @@
     <link name="root_link">
     </link>
+    <link name="base_footprint">
+    </link>
     <link name="base_link">
         <visual>
@@ -65,4 +67,9 @@
     <joint name="root_to_base" type="fixed">
         <parent link="root_link"/>
+        <child link="base_footprint"/>
+        <origin xyz="0 0 0" rpy="0 0 0" />
+    </joint>
+    <joint name="base_footprint_to_base_link" type="fixed">
+        <parent link="base_footprint"/>
         <child link="base_link"/>
         <origin xyz="0 0 0" rpy="0 0 0" />
@@ -139,19 +146,14 @@
     <xacro:rim_macro name="back" xyz="-0.072 0 0" rpy="1.570796326794896 0 1.570796326794896"/>
     <gazebo>
-        <plugin
-        filename="ignition-gazebo-velocity-control-system"
-        name="gz::sim::systems::VelocityControl">
-        </plugin>
-        <plugin filename="ignition-gazebo-joint-state-publisher-system"
-        name="ignition::gazebo::systems::JointStatePublisher">
-        </plugin>
-        <!-- ign topic -t "/model/{bot_name}/joint/arm_base/cmd_vel" -m ignition.msgs.Double -p "data: 10.0" -->
-        <plugin filename="ignition-gazebo-joint-controller-system"
-        name="gz::sim::systems::JointController">
-        <joint_name>arm_base</joint_name>
-        </plugin>
-        <plugin filename="ignition-gazebo-joint-controller-system"
-        name="gz::sim::systems::JointController">
-        <joint_name>arm_elbow</joint_name>
+        <plugin filename="libgazebo_ros_planar_move.so"
+                name="gazebo_ros_planar_move">
+            <ros>
+                <remapping>cmd_vel:=/cmd_vel</remapping>
+            </ros>
+            <update_rate>100</update_rate>
+            <publish_odom>true</publish_odom>
+            <publish_odom_tf>true</publish_odom_tf>
+            <odometry_frame>odom</odometry_frame>
+            <robot_base_frame>base_footprint</robot_base_frame>
         </plugin>
     </gazebo>

Commit message: Control joystick edit

File: description/main_core.xacro (robot description, xacro)
@@ -44,6 +44,4 @@
     <link name="root_link">
     </link>
-    <link name="base_footprint">
-    </link>
     <link name="base_link">
         <visual>
@@ -67,9 +65,4 @@
     <joint name="root_to_base" type="fixed">
         <parent link="root_link"/>
-        <child link="base_footprint"/>
-        <origin xyz="0 0 0" rpy="0 0 0" />
-    </joint>
-    <joint name="base_footprint_to_base_link" type="fixed">
-        <parent link="base_footprint"/>
         <child link="base_link"/>
         <origin xyz="0 0 0" rpy="0 0 0" />
@@ -152,8 +145,4 @@
             </ros>
             <update_rate>100</update_rate>
-            <publish_odom>true</publish_odom>
-            <publish_odom_tf>true</publish_odom_tf>
-            <odometry_frame>odom</odometry_frame>
-            <robot_base_frame>base_footprint</robot_base_frame>
         </plugin>
     </gazebo>

Commit message: Transform fix - Odom and Base_footpritn

File: description/main_core.xacro (robot description, xacro)
@@ -42,4 +42,6 @@
     </xacro:macro>
     <!-- Root link starts from here -->
+    <link name="base_footprint">
+    </link>
     <link name="root_link">
     </link>
@@ -63,4 +65,9 @@
         </inertial>
     </link>
+    <joint name="footprint_to_root" type="fixed">
+        <parent link="base_footprint"/>
+        <child link="root_link"/>
+        <origin xyz="0 0 0" rpy="0 0 0" />
+    </joint>
     <joint name="root_to_base" type="fixed">
         <parent link="root_link"/>
